Commit message: I fixed a few issues with the hopper robot's joints and foot. It looks much better now

File: RL/gym-hopping_robot/gym_hopping_robot/envs/hopping_robot/urdf/hopping_robot.urdf (robot description, URDF)
Before this commit: robot hopping_robot, 3 links, 2 joints
Links:
- link foot: geometry collision box size=0.25 0.6 0.05; visual box size=0.25 0.6 0.05
- link torso: geometry collision box size=0.4 0.4 0.4; visual box size=0.4 0.4 0.4
Joints:
- joint leg_foot: origin xyz=0.0 -0.125 -0.525 rpy=0 0 0 -> xyz=0.0 0.0 -0.525 rpy=0 0 0
- joint torso_leg: origin xyz=0.0 0.0 -0.675 rpy=0 0 0 -> xyz=0.0 0.0 -0.7 rpy=0 0 0

File: RL/gym-hopping_robot/gym_hopping_robot/envs/hopping_robot/urdf/hopping_robot.xacro (robot description, xacro)
@@ -4,13 +4,13 @@
      Date: 09/29/2020   -->
 <robot name="hopping_robot" xmlns:xacro="http://ros.org/wiki/xacro">
+	<xacro:property name="torso_width" value="0.4" />
+        <xacro:property name="torso_height" value="0.4" />
+        <xacro:property name="torso_depth" value="0.4" />
+        <xacro:property name="torso_mass" value="1.0" />
 	<xacro:property name="leg_length" value="1.0" />
 	<xacro:property name="leg_radius" value="0.05"/>
 	<xacro:property name="leg_mass" value="1.0" />
-	<xacro:property name="torso_width" value="0.35" />
-	<xacro:property name="torso_height" value="0.35" />
-        <xacro:property name="torso_depth" value="0.35" />
-        <xacro:property name="torso_mass" value="1.0" />
 	<xacro:property name="foot_width" value="0.25" />
-        <xacro:property name="foot_height" value="0.25" />
+        <xacro:property name="foot_height" value="0.60" />
         <xacro:property name="foot_depth" value="0.05" />
 	<xacro:property name="foot_mass" value="1.0" />
@@ -72,8 +72,8 @@
                                 <!-- color rgba="0 255 0 0.5" / -->
                         </material>
-			<origin rpy="0 0 0" xyz="0.0 0.0 0.0"/>
+			<origin rpy="0 0 0" xyz="0.0 ${-foot_height/2} 0.0"/>
                 </visual>
                 <inertial>
-			<origin rpy="0 0 0" xyz="0.0 0.0 0.0"/>
+			<origin rpy="0 0 0" xyz="0.0 ${-foot_height/2} 0.0"/>
                         <mass value = "1.0"/>
                         <!-- Fix the inertia tag-->
@@ -83,5 +83,5 @@
                 </inertial>
                 <collision>
-			<origin rpy="0 0 0" xyz="0.0 0.0 0.0"/>
+			<origin rpy="0 0 0" xyz="0.0 ${-foot_height/2} 0.0"/>
                         <geometry>
                                 <box size="${foot_width} ${foot_height} ${foot_depth}" />
@@ -96,5 +96,5 @@
 	</joint>
 	<joint name="leg_foot" type="revolute">
-		<origin xyz="0.0 ${-foot_width/2} ${-leg_length/2 - foot_depth/2}" rpy="0 0 0" />
+		<origin xyz="0.0 0.0 ${-leg_length/2 - foot_depth/2}" rpy="0 0 0" />
 	  	<axis xyz = "1 0 0" />
 	  	<parent link="leg" />

Commit message: I added a weekly progress report section

File: RL/gym-hopping_robot/gym_hopping_robot/envs/hopping_robot/urdf/hopping_robot.urdf (robot description, URDF)
Before this commit: robot hopping_robot, 3 links, 2 joints
Links:
- removed link leg
- added link link1, mass 1.0; collision cylinder length=0.4 radius=0.05; visual cylinder length=0.4 radius=0.05
- added link link2, mass 1.0; collision cylinder length=0.4 radius=0.05; visual cylinder length=0.4 radius=0.05
- added link link3, mass 1.0; collision cylinder length=0.4 radius=0.05; visual cylinder length=0.4 radius=0.05
Joints:
- added joint link1_link2: type revolute, parent link1, child link2, origin xyz=0.0 0.0 -0.2 rpy=0 0 0, axis 1 0 0, limit lower=-1.57 upper=1.57 effort=10 velocity=1.0
- added joint link2_link3: type revolute, parent link2, child link3, origin xyz=0.0 0.0 -0.4 rpy=0 0 0, axis 1 0 0, limit lower=-1.57 upper=1.57 effort=10 velocity=1.0
- joint leg_foot: origin xyz=0.0 0.0 -0.525 rpy=0 0 0 -> xyz=0.0 0.0 -0.425 rpy=0 0 0; parent leg -> link3
- joint torso_leg: child leg -> link1; origin xyz=0.0 0.0 -0.7 rpy=0 0 0 -> xyz=0.0 0.0 -0.4 rpy=0 0 0

File: RL/gym-hopping_robot/gym_hopping_robot/envs/hopping_robot/urdf/hopping_robot.xacro (robot description, xacro)
@@ -8,7 +8,13 @@
         <xacro:property name="torso_depth" value="0.4" />
         <xacro:property name="torso_mass" value="1.0" />
-	<xacro:property name="leg_length" value="1.0" />
-	<xacro:property name="leg_radius" value="0.05"/>
-	<xacro:property name="leg_mass" value="1.0" />
+	<xacro:property name="link1_length" value="0.4" />
+	<xacro:property name="link1_radius" value="0.05"/>
+	<xacro:property name="link1_mass" value="1.0" />
+	<xacro:property name="link2_length" value="0.4" />
+        <xacro:property name="link2_radius" value="0.05"/>
+        <xacro:property name="link2_mass" value="1.0" />
+	<xacro:property name="link3_length" value="0.4" />
+        <xacro:property name="link3_radius" value="0.05"/>
+        <xacro:property name="link3_mass" value="1.0" />
 	<xacro:property name="foot_width" value="0.25" />
         <xacro:property name="foot_height" value="0.60" />
@@ -21,5 +27,5 @@
 			</geometry>
 			<material name="gray">
-				<!-- color rgba="255 0 0 0.75" / -->
+				<!-- color rgba="255 0 0 0.75" /-->
 			</material>
 			<origin rpy="0 0 0" xyz="0.0 0.0 0.0"/>
@@ -40,11 +46,11 @@
 		</collision>
         </link>
-	<link name="leg">
+	<link name="link1">
 		 <visual>
                         <geometry>
-				 <cylinder length="${leg_length}" radius="${leg_radius}"/>
+				 <cylinder length="${link1_length}" radius="${link1_radius}"/>
                         </geometry>
                         <material name="gray">
-                                <!-- color rgba="0 0 255 0.4" / -->
+                                <!-- color rgba="0 255 0 0.4" / -->
                         </material>
 			<origin rpy="0 0 0" xyz="0 0 0"/>
@@ -53,15 +59,63 @@
 			<origin rpy="0 0 0" xyz="0 0 0"/>
                         <mass value = "1.0"/>
-			<inertia ixx="${ (1.0/12.0) * leg_mass * leg_length * leg_length}"
-				 iyy="${ (1.0/12.0) * leg_mass * leg_length * leg_length}"
-				 izz="${ (1.0/12.0) * leg_mass * leg_length * leg_length}" />
+			<inertia ixx="${ (1.0/12.0) * link1_mass * link1_length * link1_length}"
+				 iyy="${ (1.0/12.0) * link1_mass * link1_length * link1_length}"
+				 izz="${ (1.0/12.0) * link1_mass * link1_length * link1_length}" />
                 </inertial>
                 <collision>
 			<origin rpy="0 0 0" xyz="0 0 0"/>
                         <geometry>
-                        	<cylinder length="${leg_length}" radius="${leg_radius}"/>
+                        	<cylinder length="${link1_length}" radius="${link1_radius}"/>
                         </geometry>
                 </collision>
 	</link>
+	 <link name="link2">
+                 <visual>
+                        <geometry>
+                                 <cylinder length="${link2_length}" radius="${link2_radius}"/>
+                        </geometry>
+                        <material name="gray">
+                                <!-- color rgba="233 0 255 0.4" / -->
+                        </material>
+			<origin rpy="0 0 0" xyz="0 0 ${-link2_length/2}"/>
+                </visual>
+                <inertial>
+                        <origin rpy="0 0 0" xyz="0 0 ${-link2_length/2}"/>
+                        <mass value = "1.0"/>
+                        <inertia ixx="${ (1.0/12.0) * link2_mass * link2_length * link2_length}"
+                                 iyy="${ (1.0/12.0) * link2_mass * link2_length * link2_length}"
+                                 izz="${ (1.0/12.0) * link2_mass * link2_length * link2_length}" />
+                </inertial>
+                <collision>
+                        <origin rpy="0 0 0" xyz="0 0 ${-link1_length/2}"/>
+                        <geometry>
+                                <cylinder length="${link2_length}" radius="${link2_radius}"/>
+                        </geometry>
+                </collision>
+	</link>
+	<link name="link3">
+                 <visual>
+                        <geometry>
+                                 <cylinder length="${link3_length}" radius="${link3_radius}"/>
+                        </geometry>
+                        <material name="gray">
+                                <!-- color rgba="0 0 255 0.4"/ -->
+                        </material>
+			<origin rpy="0 0 0" xyz="0 0 ${-link3_length/2}"/>
+                </visual>
+                <inertial>
+			<origin rpy="0 0 0" xyz="0 0 ${-link3_length/2}"/>
+                        <mass value = "1.0"/>
+                        <inertia ixx="${ (1.0/12.0) * link3_mass * link3_length * link3_length}"
+                                 iyy="${ (1.0/12.0) * link3_mass * link3_length * link3_length}"
+                                 izz="${ (1.0/12.0) * link3_mass * link3_length * link3_length}" />
+                </inertial>
+                <collision>
+			<origin rpy="0 0 0" xyz="0 0 ${-link2_length/2}"/>
+                        <geometry>
+                                <cylinder length="${link3_length}" radius="${link3_radius}"/>
+                        </geometry>
+                </collision>
+        </link>
 	<link name="foot">
 		<visual>
@@ -91,12 +145,28 @@
 	<joint name="torso_leg" type="fixed">
 		<parent link="torso"/>
-                <child link="leg"/>
-		<origin rpy="0 0 0" xyz="0.0 0.0 ${-leg_length/2 - torso_depth/2}"/>
+                <child link="link1"/>
+		<origin rpy="0 0 0" xyz="0.0 0.0 ${-link1_length/2 - torso_depth/2}"/>
 		<axis xyz="0 0 0"/>
 	</joint>
+	<joint name="link1_link2" type="revolute">
+                <origin xyz="0.0 0.0 ${-link1_length/2}" rpy="0 0 0" />
+                <axis xyz = "1 0 0" />
+                <parent link="link1" />
+                <child link="link2" />
+                <!-- What to set these to? -->
+                <limit velocity="1.0" effort="10" lower="-1.57" upper="1.57"/>
+	</joint>
+	<joint name="link2_link3" type="revolute">
+		<origin xyz="0.0 0.0 ${-link2_length}" rpy="0 0 0" />
+                <axis xyz = "1 0 0" />
+                <parent link="link2" />
+                <child link="link3" />
+                <!-- What to set these to? -->
+                <limit velocity="1.0" effort="10" lower="-1.57" upper="1.57"/>
+        </joint>
 	<joint name="leg_foot" type="revolute">
-		<origin xyz="0.0 0.0 ${-leg_length/2 - foot_depth/2}" rpy="0 0 0" />
+		<origin xyz="0.0 0.0 ${-link3_length - foot_depth/2}" rpy="0 0 0" />
 	  	<axis xyz = "1 0 0" />
-	  	<parent link="leg" />
+	  	<parent link="link3" />
 		<child link="foot" />
 		<!-- What to set these to? -->
@@ -110,3 +180,17 @@
                 <mechanicalReduction>50</mechanicalReduction>
         </transmission>
+	<transmission name="link1_link2_trans" type="transmission_interface/SimpleTransmission">
+                <joint name="link1_link2_trans" />
+                <actuator name="link1_link2_trans"/>
+                <!-- What to set these to? -->
+                <motorInertia>0.0000049</motorInertia>
+                <mechanicalReduction>50</mechanicalReduction>
+        </transmission>
+	<transmission name="link2_link3_trans" type="transmission_interface/SimpleTransmission">
+                <joint name="link2_link3_trans" />
+                <actuator name="link2_link3_trans"/>
+                <!-- What to set these to? -->
+                <motorInertia>0.0000049</motorInertia>
+                <mechanicalReduction>50</mechanicalReduction>
+        </transmission>
 </robot>
